File: hardware/robot-board/robot-board.kicad_sch (KiCad schematic)
At the start: 110 parts, among them J1 1x8_Pin, J10 1x2_Screw, J11 1x2_Screw, J2 Barrel_Jack, J3 USB_C_Receptacle_USB2.0_14P, J4 Conn_01x03_Pin, J5 Conn_01x03_Pin, J6 Conn_01x03_Pin, J7 Conn_01x03_Pin, J8 1x2_Screw, J9 1x2_Screw, Q1 BSS138, Q2 BSS138, Q3 BSS138, Q4 BSS138, SW1 SW_SPST, U1 ESP32-S3-WROOM-1, U2 LMR51450, U3 LMR51450, U5 TPS552892, U6 DRV8835, U7 DRV8835, U8 TVS1400DRV

Commit message: schematic basically done
Parts:
- C1, C18, C2, C3, C4: JLC P/N (none) -> C307423
- C10, C9: JLC P/N (none) -> C107005
- C11, C13: JLC P/N (none) -> C140782
- C12, C14: footprint Capacitor_SMD:C_0402_1005Metric -> Capacitor_SMD:C_1206_3216Metric; JLC P/N (none) -> C342307
- C15: JLC P/N (none) -> C315248
- C16, C17, C26, C27, C30, C33: JLC P/N (none) -> C105226
- C19, C20, C21, C22, C23, C24, C25, C28, C29, C5, C6, C7, C8: JLC P/N (none) -> C1525
- C31: JLC P/N (none) -> C106200
- C32: JLC P/N (none) -> C106208
- F1: JLC P/N (none) -> C210842
- J1: JLC P/N (none) -> C2883805
- J3: JLC P/N (none) -> C2988369
- J4, J5, J6, J7: JLC P/N (none) -> C5160786
- R1, R25, R3: JLC P/N (none) -> C51048211
- R10, R11, R12, R13, R14, R7, R8, R9: JLC P/N (none) -> C105871
- R15, R16: JLC P/N (none) -> C25905
- R17, R18, R19, R21, R22, R26, R27, R28, R29, R30: JLC P/N (none) -> C2909363
- R20: JLC P/N (none) -> C163453
- R23: JLC P/N (none) -> C705780
- R24: JLC P/N (none) -> C326730
- R31: JLC P/N (none) -> C326733
- R32: footprint Resistor_SMD:R_0603_1608Metric -> Resistor_SMD:R_0805_2012Metric; JLC P/N (none) -> C728268
- R33: footprint Resistor_SMD:R_0603_1608Metric -> Resistor_SMD:R_0402_1005Metric; JLC P/N (none) -> C852841
- R34: footprint Resistor_SMD:R_0603_1608Metric -> Resistor_SMD:R_0402_1005Metric; JLC P/N (none) -> C852492
- R4: JLC P/N (none) -> C855669
- R5, R6: footprint Resistor_SMD:R_0603_1608Metric -> Resistor_SMD:R_0402_1005Metric; JLC P/N (none) -> C110776
- SW1: JLC P/N (none) -> C116647
- TP1, TP2, TP3, TP4, TP5: now left out of the parts list
- U1: JLC P/N (none) -> C2913197
- U2, U3: JLC P/N (none) -> C5782413
- U4: renamed from U8; JLC P/N (none) -> C1975229
Connections:
- net +3V3: no longer U1.3 (EN)
- net AGND: now also C1.1, C2.1, C3.1, C4.1, C5.1, C6.1
- net EN: now also U1.3 (EN)
- no-connect marks 9 -> 10
Other:
- note added: "Note that C20 should be placed close to ADC1"
- note removed: "Note that C19 should be placed close to ADC1"
- moved on the sheet: C31

Commit message: BOM and changed footprints
Parts:
- SW1: footprint random-keyboard-parts:SKQGADE010 -> footprints:SW_Push_SPST_TS-1088; JLC P/N C116647 -> C720477
Changed lines of the file:
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@@
 			)
 		)
-		(property "Footprint" "random-keyboard-parts:SKQGADE010"
+		(property "Footprint" "footprints:SW_Push_SPST_TS-1088"
 			(at 26.67 113.03 0)
 			(effects
@@
 			)
 		)
-		(property "JLC P/N" "C116647"
+		(property "JLC P/N" "C720477"
 			(at 26.67 113.03 0)
 			(effects

Commit message: bnyahaj
bnyahaj
Other:
- note added: "ESP32-S3-WROOM-1-N4"
- note removed: "ESP32-S3-WROOM"
