File: hardware/robot-board/robot-board.kicad_sch (KiCad schematic)
At the start: 128 parts, among them J1 1x8_Pin, J10 1x2_Screw, J11 1x2_Screw, J2 Barrel_Jack, J3 USB_C_Receptacle_USB2.0_14P, J4 Conn_01x03_Pin, J5 Conn_01x03_Pin, J6 Conn_01x03_Pin, J7 Conn_01x03_Pin, J8 1x2_Screw, J9 1x2_Screw, Q1 BSS138, Q2 BSS138, Q3 BSS138, Q4 BSS138, Q5 BSS138, Q6 BSS138, Q7 BSS138, Q8 BSS138, SW1 SW_SPST, U1 ESP32-S3-WROOM-1, U10 XL-SA3391SRWC, U2 LMR51450, U3 LMR51450, U4 TVS1400DRV, U5 TPS552892, U6 DRV8835, U7 DRV8835, U9 STP08CP05M

Commit message: layout!
Parts:
- removed D11: LF5, LED_SMD:LED_1206_3216Metric, symbol Device:LED
- removed D5: LF1, LED_SMD:LED_1206_3216Metric, symbol Device:LED
- removed D9: LF3, LED_SMD:LED_1206_3216Metric, symbol Device:LED
- removed J1: 1x8_Pin, Connector_PinHeader_2.54mm:PinHeader_1x08_P2.54mm_Vertical_SMD_Pin1Left, symbol Connector:Conn_01x08_Pin
- removed R21, R28, R30: 5.1R, Resistor_SMD:R_0402_1005Metric, symbol Device:R_Small
- added J1: Conn_01x09_Pin, Connector_PinHeader_2.54mm:PinHeader_1x09_P2.54mm_Vertical_SMD_Pin1Left, symbol Connector:Conn_01x09_Pin
- added NT1, NT2, NT3: NetTie_2, NetTie:NetTie-2_SMD_Pad0.5mm, symbol Device:NetTie_2
- added R16: 180R, Resistor_SMD:R_0402_1005Metric, symbol Device:R_Small
- added R42, R43: 22R, Resistor_SMD:R_0402_1005Metric, symbol Device:R_Small
- BZ1: footprint (none) -> Buzzer_Beeper:MLT-7525; JLC P/N (none) -> C95299
- D1: renamed from D12; footprint (none) -> Diode_SMD:D_SOD-123; JLC P/N (none) -> C82544
- J10, J11, J8, J9: footprint RedRobotFootprints:ScrewTerminalP3.5mm -> footprints:CONN2_2060-452&slash_998-404_WAG; JLC P/N C695629 -> C2765055
- J4, J5, J6, J7: footprint Connector_PinHeader_2.54mm:PinHeader_1x02_P2.54mm_Vertical_SMD_Pin1Right -> Connector_PinHeader_2.54mm:PinHeader_1x03_P2.54mm_Vertical_SMD_Pin1Right
- R1: renamed from R43; footprint (none) -> Resistor_SMD:R_0402_1005Metric; JLC P/N (none) -> C25905
- R34: renamed from R42; footprint (none) -> Resistor_SMD:R_0402_1005Metric; JLC P/N (none) -> C138002
- R35: renamed from R41; footprint (none) -> Resistor_SMD:R_0402_1005Metric; JLC P/N (none) -> C138002
- R36: renamed from R40; footprint (none) -> Resistor_SMD:R_0402_1005Metric; JLC P/N (none) -> C138002
- R37: renamed from R39; footprint (none) -> Resistor_SMD:R_0402_1005Metric; JLC P/N (none) -> C138002
- R38: footprint (none) -> Resistor_SMD:R_0402_1005Metric; JLC P/N (none) -> C138002
- R39: renamed from R37; footprint (none) -> Resistor_SMD:R_0402_1005Metric; JLC P/N (none) -> C138002
- R40: renamed from R36; footprint (none) -> Resistor_SMD:R_0402_1005Metric; JLC P/N (none) -> C138002
- R41: renamed from R35; footprint (none) -> Resistor_SMD:R_0402_1005Metric; JLC P/N (none) -> C138002
- U8: renamed from U10; footprint (none) -> Display_7Segment:XL-SA3391SRWC
- U9: JLC P/N (none) -> C2678582
- renumbered D1 to D2, D2 to D3, D3 to D4, D4 to D5, D7 to D6, D6 to D7, D10 to D8, D8 to D9, Q8 to Q5, Q5 to Q6, Q6 to Q7, Q7 to Q8, R9 to R10, R10 to R11, R11 to R12, R12 to R13, R13 to R14, R14 to R15, R15 to R17, R16 to R18, R17 to R19, R1 to R2, R18 to R20, R19 to R21, R20 to R22, R26 to R23, R22 to R24, R23 to R25, R24 to R26, R25 to R27, R29 to R28, R27 to R29, R2 to R3, R31 to R30, R32 to R31, R33 to R32, R34 to R33, R3 to R4, R4 to R5, R5 to R6, R6 to R7, R7 to R8, R8 to R9, TP6 to TP1, TP1 to TP2, TP2 to TP3, TP3 to TP4, TP4 to TP5, TP5 to TP6
Connections:
- net LF0_LED is gone; now on net LFL_LED: R21.1
- net LF2_LED is gone; now on net LFC_LED: R23.1
- net LF4_LED is gone; now on net LFR_LED: R28.1
- net +3V3: now also J1.2 (Pin_2)
- net AGND: now also NT1.1, NT2.1; no longer C1.1, C11.1, C12.1, C13.1, C14.1, C16.1, C17.1, C19.1, C2.1, C25.1, C26.1, C27.1, C3.1, C30.1, C33.1, C4.1, C5.1, C6.1, U2.13 (PGND), U3.13 (PGND), U5.9 (PGND)
- net BUZZER: now also R16.1; no longer Q5.1 (G)
- net GND: now also J1.1 (Pin_1), NT3.1
- net LF0: now also J1.3 (Pin_3)
- net LF1: now also J1.4 (Pin_4)
- net LF2: now also J1.5 (Pin_5)
- net LF3: now also J1.6 (Pin_6)
- net LF4: now also J1.7 (Pin_7)
- net LF5: now also J1.8 (Pin_8)
- net LF_LEDCTRL: now also U1.36 (RXD0), J1.9 (Pin_9); no longer U1.22 (IO14)
- net MOTOR2_EN: now also U1.22 (IO14); no longer U1.36 (RXD0)
- net USB_DM: now also R42.2; no longer J3.A7 (D-), J3.B7 (D-)
- net USB_DP: now also R43.2; no longer J3.A6 (D+), J3.B6 (D+)
- new net: Q5.1 (G), R16.2
- new net: J3.A7 (D-), J3.B7 (D-), R42.1
- new net: J3.A6 (D+), J3.B6 (D+), R43.1
- new net PGND: C1.1, C11.1, C12.1, C13.1, C14.1, C16.1, C17.1, C19.1, C2.1, C25.1, C26.1, C27.1, C3.1, C30.1, C33.1, C4.1, C5.1, C6.1, NT1.2, NT2.2, NT3.2, U2.13 (PGND), U3.13 (PGND), U5.9 (PGND)
Other:
- note added: "Note R34-R41 are all 33 Ohm resistors"
- note removed: "Note R35-R42 are all 33 Ohm resistors"
- moved on the sheet: C20, D4, D6, D8, Q6, Q7, Q8, R21, R23, R26, R27, R28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

Commit message: fixed some stuff
Connections:
- net GND: now also U6.13 (GND), U7.13 (GND); no longer J3.S1 (SHIELD)
- no-connect marks 12 -> 13
Changed lines of the file:
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@@
 	)
 	(no_connect
+		(at 125.73 195.58)
+	)
+	(no_connect
 		(at 46.99 143.51)
 	)
@@
 		(pin "3"
 		)
+		(pin "13"
+		)
 		(instances
 			(project "robot-board"
@@
 		(pin "3"
 		)
+		(pin "13"
+		)
 		(instances
 			(project ""
@@
 					(unit 1)
 				)
-			)
-		)
-	)
-	(symbol
-		(lib_id "power:GND")
-		(at 125.73 195.58 0)
-		(unit 1)
-		(exclude_from_sim no)
-		(in_bom yes)
-		(on_board yes)
-		(dnp no)
-		(fields_autoplaced yes)
-		(property "Reference" "#PWR028"
-			(at 125.73 201.93 0)
-			(effects
-				(font
-					(size 1.27 1.27)
-				)
-				(hide yes)
-			)
-		)
-		(property "Value" "GND"
-			(at 125.73 200.66 0)
-			(effects
-				(font
-					(size 1.27 1.27)
-				)
-			)
-		)
-		(property "Footprint" ""
-			(at 125.73 195.58 0)
-			(effects
-				(font
-					(size 1.27 1.27)
-				)
-				(hide yes)
-			)
-		)
-		(property "Datasheet" ""
-			(at 125.73 195.58 0)
-			(effects
-				(font
-					(size 1.27 1.27)
-				)
-				(hide yes)
-			)
-		)
-		(property "Description" "Power symbol creates a global label with name \"GND\" , ground"
-			(at 125.73 195.58 0)
-			(effects
-				(font
-					(size 1.27 1.27)
-				)
-				(hide yes)
-			)
-		)
-		(pin "1"
-		)
-		(instances
-			(project ""
-				(path "/3adacf52-553b-4591-a9be-9572be717553"
-					(reference "#PWR028")
-					(unit 1)
-				)

Commit message: who up roboing their club
Parts:
- J2: footprint Connector_BarrelJack:BarrelJack_Horizontal -> Connector_BarrelJack:BarrelJack_CLIFF_FC681465S_SMT_Horizontal; JLC P/N C136744 -> C114916
Changed lines of the file:
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@@
 			)
 		)
-		(property "Footprint" "Connector_BarrelJack:BarrelJack_Horizontal"
+		(property "Footprint" "Connector_BarrelJack:BarrelJack_CLIFF_FC681465S_SMT_Horizontal"
 			(at 129.286 139.7 0)
 			(effects
@@
 			)
 		)
-		(property "Description" ""
+		(property "Description" "DC Barrel Jack with an internal switch"
 			(at 128.27 140.97 0)
 			(effects
@@
 			)
 		)
-		(property "JLC P/N" "C136744"
+		(property "JLC P/N" "C114916"
 			(at 128.27 140.97 0)
 			(effects

Commit message: gerbers n stuff hi hi
Parts:
- removed TP1: D0, TestPoint:TestPoint_THTPad_2.0x2.0mm_Drill1.0mm, symbol Connector:TestPoint
- added D10: D_Small, Diode_SMD:D_SOD-123, symbol Device:D_Small
- added JP1: SolderJumper_2_Open, Jumper:SolderJumper-2_P1.3mm_Open_Pad1.0x1.5mm, symbol Jumper:SolderJumper_2_Open
- added R44: 5.1k, Resistor_SMD:R_0402_1005Metric, symbol Device:R_Small
- added SW2: SW_SPST, footprints:SW_Push_SPST_TS-1088, symbol Switch:SW_SPST
- J1: JLC P/N C41417348 -> C49423356
Connections:
- net +3V3: now also R44.1
- net +5V: now also JP1.2 (B)
- net GND: now also SW2.2 (B)
- net LBAT_LED: now also U1.9 (IO16); no longer U1.27 (IO0)
- net at J3.A4 (VBUS), J3.A9 (VBUS), J3.B4 (VBUS)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: now also D10.2 (A)
- new net: D10.1 (K), JP1.1 (A)
- new net BS: R44.2, SW2.1 (A), U1.27 (IO0)
- no-connect marks 13 -> 11
Other:
- note added: "Boot Select"

Commit message: fixed the thingies
Parts:
- C11, C13: footprint Capacitor_SMD:C_0402_1005Metric -> Capacitor_SMD:C_0603_1608Metric
Changed lines of the file:
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@@
 			)
 		)
-		(property "Footprint" "Capacitor_SMD:C_0402_1005Metric"
+		(property "Footprint" "Capacitor_SMD:C_0603_1608Metric"
 			(at 97.79 135.89 0)
 			(effects
@@
 			)
 		)
-		(property "Footprint" "Capacitor_SMD:C_0402_1005Metric"
+		(property "Footprint" "Capacitor_SMD:C_0603_1608Metric"
 			(at 106.68 135.89 0)
 			(effects

Commit message: fixed footprint/part mismatch
Parts:
- R6, R7: JLC P/N C110776 -> C2906864
- U6, U7: JLC P/N C82045 -> C129328
Changed lines of the file:
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@@
 			)
 		)
-		(property "JLC P/N" "C82045"
+		(property "JLC P/N" "C129328"
 			(at 236.22 101.6 0)
 			(effects
@@
 			)
 		)
-		(property "JLC P/N" "C110776"
+		(property "JLC P/N" "C2906864"
 			(at 90.17 177.8 0)
 			(effects
@@
 			)
 		)
-		(property "JLC P/N" "C82045"
+		(property "JLC P/N" "C129328"
 			(at 236.22 74.93 0)
 			(effects
@@
 			)
 		)
-		(property "JLC P/N" "C110776"
+		(property "JLC P/N" "C2906864"
 			(at 90.17 135.89 0)
 			(effects
