File: hardware/robot-board/robot-board.kicad_pcb (KiCad board)
At the start: 4 copper layers, 69 x 99 mm, 129 parts, among them J1 Conn_01x09_Pin, J10 1x2_Screw, J11 1x2_Screw, J2 Barrel_Jack, J3 USB_C_Receptacle_USB2.0_14P, J4 Conn_01x03_Pin, J5 Conn_01x03_Pin, J6 Conn_01x03_Pin, J7 Conn_01x03_Pin, J8 1x2_Screw, J9 1x2_Screw, Q1 BSS138, Q2 BSS138, Q3 BSS138, Q4 BSS138, Q5 BSS138, Q6 BSS138, Q7 BSS138, Q8 BSS138, SW1 SW_SPST, U1 ESP32-S3-WROOM-1, U2 LMR51450, U3 LMR51450, U4 TVS1400DRV, U5 TPS552892, U6 DRV8835, U7 DRV8835, U8 XL-SA3391SRWC, U9 STP08CP05M

Commit message: fixed some stuff
Parts:
- D2: renamed from LOW BATT
- moved C15 24.8 mm to (66.2, 72.5)
- moved F1 24.8 mm to (72.4, 70.8)
- moved J2 24.8 mm to (72.4, 63.2)
- moved U4 24.8 mm to (68.1, 70.9)
- moved J1 15.0 mm to (89.7, 57.7)
- moved R21 14.3 mm to (96.0, 64.0)
- moved D4 14.3 mm to (99.5, 64.0)
- moved D6 14.3 mm to (99.4, 69.2)
- moved D8 14.3 mm to (99.4, 74.4)
- moved R23 14.3 mm to (95.9, 69.3)
- moved R28 14.3 mm to (95.9, 74.5)
- moved R17 2.40 mm to (47.4, 142.6)
- moved R18 2.40 mm to (42.0, 142.6)
- moved J3 2.40 mm to (44.7, 148.3)
- renumbered COMMS to D3, LEFT to D4, POWER to D5, CENTER to D6, TX to D7, RIGHT to D8, RX to D9, NC to TP1, BMS_D0 to TP2, BMS_D1 to TP3, BMS_D2 to TP4, BMS_SDI to TP5, BMS_CLK to TP6
Connections:
- J10 pad 1: /M2+ -> /M2-
- J3 pad S1: GND -> unconnected-(J3-SHIELD-PadS1)_2
Routing:
- net Vprot: track 117.9 -> 90.3 mm
- net +3V3: track 221.5 -> 236.5 mm
- net /LF3: track 50.8 -> 65.1 mm
- net /LF4: track 53.6 -> 67.8 mm
- net /LF0: track 55.7 -> 69.9 mm
- net /LF5: track 49.8 -> 64.0 mm
- net /LF1: track 51.9 -> 66.1 mm
- net /LF2: track 54.6 -> 68.9 mm
- net /LF_LEDCTRL: track 53.3 -> 66.8 mm
- net /LFL_LED: track 64.6 -> 77.3 mm
- net /LFR_LED: track 56.7 -> 67.0 mm
- net GND: track 21.4 -> 30.8 mm, vias 67 -> 68
- net /LFC_LED: track 60.5 -> 68.7 mm
- net +BATT: track 14.3 -> 15.5 mm
- net Net-(J3-D+-PadA6): track 31.5 -> 30.5 mm
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Other:
- board text added: "BMS_CLK"
- board text added: "BMS_D0"
- board text added: "BMS_D1"
- board text added: "BMS_D2"
- board text added: "BMS_SDI"
- board text added: "CENTER"
- board text added: "COMMS"
- board text added: "LEFT"
- board text added: "LOW BATT"
- board text added: "NC"
- board text added: "POWER"
- board text added: "RIGHT"
- board text added: "RX"
- board text added: "TX"

Commit message: who up roboing their club
Parts:
- J2: footprint Connector_BarrelJack:BarrelJack_Horizontal -> Connector_BarrelJack:BarrelJack_CLIFF_FC681465S_SMT_Horizontal
- moved J2 5.85 mm to (70.2, 57.8)
Routing:
- net +BATT: track 15.5 -> 25.4 mm
- net +3V3: track 236.5 -> 237.0 mm, vias 8 -> 10
- net GND: vias 68 -> 67

Commit message: gerbers n stuff hi hi
Parts:
- removed TP1: D0, TestPoint:TestPoint_THTPad_2.0x2.0mm_Drill1.0mm
- added D10: D_Small, Diode_SMD:D_SOD-123, F.Cu at (48.1, 87.5)
- added G***: LOGO, LOGO, B.Cu at (95.0, 136.3)
- added G***: LOGO, LOGO, B.Cu at (74.1, 136.7)
- added G***: LOGO, LOGO, B.Cu at (93.0, 73.1)
- added G***: LOGO, LOGO, B.Cu at (52.3, 136.7)
- added JP1: SolderJumper_2_Open, Jumper:SolderJumper-2_P1.3mm_Open_Pad1.0x1.5mm, F.Cu at (51.8, 86.8)
- added R44: 5.1k, Resistor_SMD:R_0402_1005Metric, F.Cu at (41.9, 87.8)
- added SW2: SW_SPST, footprints:SW_Push_SPST_TS-1088, F.Cu at (44.2, 90.5)
Connections:
- J3 pad A4: unconnected-(J3-VBUS-PadA4)_3 -> Net-(D10-A)
- J3 pad A9: unconnected-(J3-VBUS-PadA4)_1 -> Net-(D10-A)
- J3 pad B4: unconnected-(J3-VBUS-PadA4)_2 -> Net-(D10-A)
- J3 pad B9: unconnected-(J3-VBUS-PadA4) -> Net-(D10-A)
- U1 pad 27: /LBAT_LED -> /BS
- U1 pad 9: Net-(U1-IO16) -> /LBAT_LED
Routing:
- net Net-(D10-A): track 0.00 -> 68.0 mm, vias 0 -> 2
- net /BS: track 0.00 -> 22.0 mm, vias 0 -> 2
- net /LBAT_LED: track 54.0 -> 74.7 mm, vias 4 -> 6
- net Net-(U1-IO16): track 4.68 -> 0.00 mm
- net +3V3: track 237.0 -> 240.3 mm
- net /LFL_LED: track 77.3 -> 74.9 mm
- net +5V: track 176.5 -> 178.9 mm
- net Net-(D10-K): track 0.00 -> 2.01 mm
- net /MOTOR0_EN: track 49.4 -> 48.5 mm
- net GND: vias 67 -> 68
Other:
- board text removed: "NC"

Commit message: fixed the thingies
Parts:
- C11, C13: footprint Capacitor_SMD:C_0402_1005Metric -> Capacitor_SMD:C_0603_1608Metric
- moved C11 0.64 mm to (50.9, 56.0)
- moved C13 0.22 mm to (50.9, 57.5)
Routing:
- net +3V3: track 240.3 -> 241.6 mm
- net PGND: track 69.1 -> 70.0 mm
