File: hardware/robot-board/robot-board.kicad_pcb (KiCad board)
At the start: 4 copper layers, 69 x 99 mm, 136 parts, among them J1 Conn_01x09_Pin, J10 1x2_Screw, J11 1x2_Screw, J2 Barrel_Jack, J3 USB_C_Receptacle_USB2.0_14P, J4 Conn_01x03_Pin, J5 Conn_01x03_Pin, J6 Conn_01x03_Pin, J7 Conn_01x03_Pin, J8 1x2_Screw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

Commit message: fixed all issues, removed LF LEDs
Parts:
- removed D4: LF0, LED_SMD:LED_1206_3216Metric
- removed D6: LF2, LED_SMD:LED_1206_3216Metric
- removed D8: LF4, LED_SMD:LED_1206_3216Metric
- removed R21, R23, R28: 5.1R, Resistor_SMD:R_0402_1005Metric
- added G***: LOGO, LOGO, F.Cu at (95.4, 70.1)
- added REF**: KiCad-Logo_6mm_SilkScreen, Symbol:KiCad-Logo_6mm_SilkScreen, B.Cu at (47.5, 58.5)
- turned U4 to 90 degrees
Connections:
- U1 pad 16: /SERVO1_PWM -> unconnected-(U1-IO46-Pad16)
- U1 pad 19: /LFC_LED -> unconnected-(U1-IO11-Pad19)
- U1 pad 20: /LFL_LED -> /SERVO1_PWM
- U1 pad 21: /LFR_LED -> /SERVO0_PWM
- U1 pad 26: /SERVO0_PWM -> unconnected-(U1-IO45-Pad26)
- U4 pad 1: +BATT -> GND
- U4 pad 2: +BATT -> GND
- U4 pad 3: +BATT -> GND
- U4 pad 4: GND -> +BATT
- U4 pad 5: GND -> +BATT
- U4 pad 6: GND -> +BATT
- U4 pad 7: +BATT -> GND
Routing:
- net /LFL_LED: track 74.9 -> 0.00 mm, vias 4 -> 0
- net /LFC_LED: track 68.7 -> 0.00 mm, vias 2 -> 0
- net /LFR_LED: track 67.0 -> 0.00 mm, vias 2 -> 0
- net +BATT: track 25.4 -> 0.91 mm
- net Vprot: track 90.3 -> 81.7 mm
- net GND: track 30.8 -> 25.2 mm
- net /SERVO1_PWM: track 50.1 -> 52.2 mm
- net /SERVO0_PWM: track 64.3 -> 62.2 mm
- net Net-(D6-A): track 1.57 -> 0.00 mm
- net Net-(D8-A): track 1.56 -> 0.00 mm
- net Net-(D4-A): track 1.52 -> 0.00 mm
- net /LBAT_LED: track 74.7 -> 73.6 mm
- net /SERVO3_PWM: track 45.1 -> 44.8 mm, vias 2 -> 0
- net /SERVO2_PWM: track 48.3 -> 48.0 mm, vias 2 -> 0
Other:
- board text removed: "CENTER"
- board text removed: "LEFT"
- board text removed: "RIGHT"
