File: hardware/robot-board/robot-board.kicad_pcb (KiCad board)
At the start: 4 copper layers, 69 x 99 mm, 136 parts, among them J1 Conn_01x09_Pin, J10 1x2_Screw, J11 1x2_Screw, J2 Barrel_Jack, J3 USB_C_Receptacle_USB2.0_14P, J4 Conn_01x03_Pin, J5 Conn_01x03_Pin, J6 Conn_01x03_Pin, J7 Conn_01x03_Pin, J8 1x2_Screw, J9 1x2_Screw, Q1 BSS138, Q2 BSS138, Q3 BSS138, Q4 BSS138, Q5 BSS138, SW1 SW_SPST, SW2 SW_SPST, SW3 SW_SPST, U1 ESP32-S3-WROOM-1, U10 MAX7219, U2 LMR51450, U3 LMR51450, U4 TVS1400DRV, U6 DRV8835, U7 DRV8835, U8 XL-SA3391SRWC, U9 74ACT125

Commit message: swapped TVS1400 for SMBJ12A
Parts:
- U4: value TVS1400DRV -> SMBJ12A; footprint Package_SON:WSON-6-1EP_2x2mm_P0.65mm_EP1x1.6mm -> Diode_SMD:D_SMB
- moved R28 4.79 mm to (87.8, 62.2), turned to 180 degrees
- moved SW3 3.43 mm to (86.1, 55.5)
- moved U4 2.74 mm to (81.8, 61.0), turned to 0 degrees
Connections:
- U4 pad 1: GND -> +BATT
Routing:
- net Net-(F1-Pad2): track 9.39 -> 7.27 mm
- net GND: vias 106 -> 107

Commit message: Added vias, updated output files
Routing:
- net GND: vias 107 -> 109
Changed lines of the file:
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@@
 	)
 	(via
+		(at 66.1924 111.506)
+		(size 0.6)
+		(drill 0.3)
+		(layers "F.Cu" "B.Cu")
+		(free yes)
+		(net "GND")
+	)
+	(via
 		(at 103.124 95.504)
 		(size 0.6)
@@
 	)
 	(via
+		(at 67.4624 109.8296)
+		(size 0.6)
+		(drill 0.3)
+		(layers "F.Cu" "B.Cu")
+		(free yes)
+		(net "GND")
+	)
+	(via
 		(at 82.804 113.538)
 		(size 0.6)
@@
 		(layer "F.Cu")
 		(hatch none 0.1)
-		(priority 30200)
+		(priority 30199)
 		(attr
 			(teardrop
@@
 		(polygon
 			(pts
-				(xy 49.105 79.805) (xy 48.905 79.805) (xy 48.88 79.93) (xy 49.005 80.056) (xy 49.13 79.93)
+				(xy 48.905 80.305) (xy 49.105 80.305) (xy 49.13 80.18) (xy 49.005 80.054) (xy 48.88 80.18)
 			)
 		)
@@
 		(layer "F.Cu")
 		(hatch none 0.1)
-		(priority 30199)
+		(priority 30200)
 		(attr
 			(teardrop
@@
 		(polygon
 			(pts
-				(xy 48.905 80.305) (xy 49.105 80.305) (xy 49.13 80.18) (xy 49.005 80.054) (xy 48.88 80.18)
+				(xy 49.105 79.805) (xy 48.905 79.805) (xy 48.88 79.93) (xy 49.005 80.056) (xy 49.13 79.93)
 			)
 		)

Commit message: moved 5V line to back
Parts:
- removed Q6: ~, Package_SO:SOIC-8_3.9x4.9mm_P1.27mm
- removed R28: 100k, Resistor_SMD:R_0603_1608Metric
- removed SW3: SW_SPST, Button_Switch_SMD:SW_SPDT_Shouhan_MSK12C02
Connections:
- F1 pad 2: Net-(F1-Pad2) -> Vprot
Routing:
- net Net-(Q6-G): track 19.5 -> 0.00 mm
- net Net-(F1-Pad2): track 7.27 -> 0.00 mm
- net GND: vias 109 -> 102
Other:
- board text added: "Revision 3 10/20/2026 Red Robot 2026"
