File: hardware/7segdisplay/7segdisplay.kicad_sch (KiCad schematic)
At the start: 19 parts, among them U2 74LS596, U3 74LS596, U4 CC56-12SURKWA

Commit message: Fixed 7segmentdisplay sch file to include version 1 and 2a and 2b
Parts:
- added GA|NMOS1, GA|NMOS2, GA|NMOS3, GA|NMOS4, GA|NMOS5, GA|NMOS6: NMOS, symbol Simulation_SPICE:NMOS
- added R10, R14, R9: 33R, symbol Device:R_Small_US
- added R11, R12, R13, R15, R16, R17, R18, R19: 220R, symbol Device:R_Small_US
- added U1, U6, U7, U9: 74LS596, symbol 74xx:74LS596
- added U5, U8: CC56-12SURKWA, Display_7Segment:CA56-12SURKWA, symbol Display_Character:CC56-12SURKWA
Connections:
- net GND: now also U2.8 (GND), U3.8 (GND), U1.8 (GND), U6.8 (GND), U7.8 (GND), U9.8 (GND)
- net QH: now also U1.14 (SER), U7.14 (SER)
- net RCLK: now also U1.12 (RCLK), U6.12 (RCLK), U7.12 (RCLK), U9.12 (RCLK)
- net SER: now also U6.9 (QH'), U9.9 (QH')
- net SRCLK: now also U1.11 (SRCLK), U6.11 (SRCLK), U7.11 (SRCLK), U9.11 (SRCLK)
- net +5V: now reaches U2.16 (VCC)
- net +5V: now also U3.16 (VCC), GA|NMOS1.3 (S), GA|NMOS2.3 (S), GA|NMOS3.3 (S), U1.16 (VCC), U6.16 (VCC), U7.16 (VCC), U9.16 (VCC)
- new net: GA|NMOS2.2 (G), U1.1 (QB)
- new net: GA|NMOS1.2 (G), U1.15 (QA)
- new net: GA|NMOS3.2 (G), U1.2 (QC)
- new net: U5.1 (e), U6.3 (QD)
- new net: U5.10 (f), U6.2 (QC)
- new net: U5.11 (a), U6.7 (QH)
- new net: R9.1, U5.12 (CC1)
- new net: U5.2 (d), U6.4 (QE)
- new net: U5.3 (DPX), U6.15 (QA)
- new net: U5.4 (c), U6.5 (QF)
- new net: U5.5 (g), U6.1 (QB)
- new net: U5.7 (b), U6.6 (QG)
- new net: R10.1, U5.8 (CC3)
- new net: R14.1, U5.9 (CC2)
- new net: GA|NMOS3.1 (D), R10.2
- new net: GA|NMOS5.1 (D), U8.9 (CC2)
- new net: GA|NMOS5.2 (G), U7.1 (QB)
- new net: R18.1, U9.1 (QB)
- new net: R19.1, U9.15 (QA)
- new net: R17.1, U9.2 (QC)
- new net: R16.1, U9.3 (QD)
- new net: R15.1, U9.4 (QE)
- new net: R13.1, U9.5 (QF)
- new net: R12.1, U9.6 (QG)
- new net: R11.1, U9.7 (QH)
- new net: GA|NMOS1.1 (D), R9.2
- new net: GA|NMOS2.1 (D), R14.2
- new net: R15.2, U8.2 (d)
- new net: R11.2, U8.11 (a)
- new net: R12.2, U8.7 (b)
- new net: GA|NMOS4.1 (D), U8.12 (CC1)
- new net: GA|NMOS4.2 (G), U7.15 (QA)
- new net: R19.2, U8.3 (DPX)
- new net: GA|NMOS6.1 (D), U8.8 (CC3)
- new net: GA|NMOS6.2 (G), U7.2 (QC)
- new net: R13.2, U8.4 (c)
- new net: R16.2, U8.1 (e)
- new net: R17.2, U8.10 (f)
- new net: R18.2, U8.5 (g)
Other:
- note added: "Version 1 (Older, likely will not use)"
- moved on the sheet: GA|NMOS, GB|NMOS, GC|NMOS, GD|NMOS, GE|NMOS, GF, GG|NMOS, GH, R1, R2, R3, R4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
