File: hardware/line-sensor/line-sensor.kicad_pcb (KiCad board)
At the start: 2 copper layers, 75.3 x 18.5 mm, 28 parts, among them J1 Conn_01x07_Socket, J2 Conn_01x02_Socket, Q1 AO3400A, U1 QRE1113GR, U2 QRE1113GR, U3 QRE1113GR, U4 QRE1113GR, U5 QRE1113GR, U6 QRE1113GR

Commit message: uhhh i hope this works, delaynie
Parts:
- J1, J2: moved to B.Cu
- turned J1 to -90 degrees
- turned J2 to 90 degrees
Routing:
- net /LED_LOW: track 0.00 -> 72.4 mm, vias 0 -> 2
- net /OUT6: track 0.00 -> 52.5 mm, vias 0 -> 3
- net /LED_ON: track 0.00 -> 48.2 mm, vias 0 -> 1
- net Net-(C2-Pad2): track 0.00 -> 44.9 mm
- net Net-(C3-Pad2): track 0.00 -> 41.8 mm, vias 0 -> 4
- net /OUT5: track 0.00 -> 41.0 mm, vias 0 -> 3
- net Net-(C1-Pad2): track 0.00 -> 39.2 mm
- net /OUT4: track 0.00 -> 32.1 mm, vias 0 -> 1
- net +3V3: track 0.00 -> 27.0 mm, vias 0 -> 6
- net GND: track 0.00 -> 26.1 mm, vias 0 -> 12
- net /OUT3: track 0.00 -> 20.7 mm, vias 0 -> 1
- net /OUT2: track 0.00 -> 13.8 mm, vias 0 -> 1
- net Net-(C5-Pad2): track 0.00 -> 12.6 mm
- net Net-(C6-Pad2): track 0.00 -> 11.1 mm
- net Net-(C4-Pad2): track 0.00 -> 10.4 mm
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- added copper zone on F.Cu, net +3V3
- added copper zone on B.Cu, net GND
